File: projects/EXP/TOP1/top/Touch_sesor.sch (KiCad schematic (older format))
At the start: 3 parts, among them J1 Conn_01x03, J2 Conn_01x03

Commit message: New library files and schematics with ESE31 and DT045 switches
Parts:
- PCB1: symbol hitesh_custom:TouchSensor -> top-rescue:TouchSensor-hitesh_custom
Changed lines of the file:
@@
 EESchema Schematic File Version 4
 LIBS:top-cache
-LIBS:pcb1-cache
 EELAYER 26 0
 EELAYER END
@@
 $EndComp
 $Comp
-L hitesh_custom:TouchSensor PCB1
+L top-rescue:TouchSensor-hitesh_custom PCB1
 U 1 1 5CC05BAC
 P 3700 1950
+AR Path="/5CC05BAC" Ref="PCB1"  Part="1"
+AR Path="/5CC0853C/5CC05BAC" Ref="PCB1"  Part="1"
 F 0 "PCB1" V 3864 1922 50  0000 R CNN
 F 1 "TouchSensor" V 3773 1922 50  0000 R CNN
