File: projects/EXP/TOP1/top/top.sch (KiCad schematic (older format))
At the start: 8 parts, among them J6 Conn_01x02, J7 Conn_01x02, J8 Conn_01x02, J9 Conn_01x02, SW1 SW_SPST, SW2 SW_SPST

Commit message: New library files and schematics with ESE31 and DT045 switches
Parts:
- removed D1: LED, Button_Switch_SMD:SW_DIP_SPSTx01_Slide_6.7x4.1mm_W6.73mm_P2.54mm_LowProfile_JPin, symbol Device:LED
- removed D2: D_Photo, LED_SMD:LED_0805_2012Metric, symbol Device:D_Photo
- removed J6, J7, J8, J9: Conn_01x02, Connector_JST:JST_EH_B02B-EH-A_1x02_P2.50mm_Vertical, symbol Connector_Generic:Conn_01x02
- removed SW1, SW2: SW_SPST, Button_Switch_SMD:SW_DIP_SPSTx01_Slide_6.7x4.1mm_W6.73mm_P2.54mm_LowProfile_JPin, symbol Switch:SW_SPST
- added P1: Digital, Socket_Arduino_Pro_Mini:Socket_Strip_Arduino_1x12, symbol Connector_Generic:Conn_01x12
- added P2: COM, Socket_Arduino_Pro_Mini:Socket_Strip_Arduino_1x06, symbol Connector_Generic:Conn_01x06
- added P3, P5: ADC, Socket_Arduino_Pro_Mini:Socket_Strip_Arduino_1x02, symbol Connector_Generic:Conn_01x02
- added P4: Analog, Socket_Arduino_Pro_Mini:Socket_Strip_Arduino_1x12, symbol Connector_Generic:Conn_01x12
Connections:
- net labels added: 0(Rx), 1(Tx), 10(**/SS), 11(**/MOSI), 12(MISO), 13(SCK), 2, 3(**), 4, 5(**), 6(**), 7, 8, 9(**), A0, A1, A2, A3, A4, A5, A6, A7, DTR, GND, RAW, Reset, VCC
- wire segments 16 -> 33
Other:
- note added: "1"
- note added: "Shield Arduino Pro Mini \n"
