File: projects/MOTBOX_TOP/limit_switch/limit_switch.kicad_pcb (KiCad board)
At the start: 2 copper layers, 10 x 12 mm, 3 parts, among them J1 Conn_02x02_Top_Bottom, SW1 SW_SPST, SW2 SW_SPST

Commit message: New library files and schematics with ESE31 and DT045 switches
Parts:
- SW1: value SW_SPST -> ESE31R11T
- SW2: value SW_SPST -> ESE31L11T
Other:
- board text added: "Need to change the foot print of Det switch"
Changed lines of the file:
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@@
   (general
     (thickness 1.6)
-    (drawings 4)
+    (drawings 5)
     (tracks 14)
     (zones 0)
@@
     (pcbplotparams
       (layerselection 0x010fc_ffffffff)
-      (usegerberextensions false)
+      (usegerberextensions true)
       (usegerberattributes false)
       (usegerberadvancedattributes false)
@@
       (outputformat 1)
       (mirror false)
-      (drillshape 1)
+      (drillshape 0)
       (scaleselection 1)
-      (outputdirectory ""))
+      (outputdirectory "Gerber/"))
   )
   (net 0 "")
@@
       (effects (font (size 1 1) (thickness 0.15)))
     )
-    (fp_text value SW_SPST (at -0.5 -4.5 270) (layer F.Fab) hide
+    (fp_text value ESE31R11T (at -0.5 -4.5 270) (layer F.Fab) hide
       (effects (font (size 1 1) (thickness 0.15)))
     )
@@
       (effects (font (size 1 1) (thickness 0.15)))
     )
-    (fp_text value SW_SPST (at -0.5 -4.5 90) (layer F.Fab) hide
+    (fp_text value ESE31L11T (at -0.5 -4.5 90) (layer F.Fab) hide
       (effects (font (size 1 1) (thickness 0.15)))
     )
@@
       (net 4 "Net-(J1-Pad2)"))
   )
+  (gr_text "Need to change the foot print of Det switch" (at 166.3 88.5) (layer Cmts.User)
+    (effects (font (size 1.5 1.5) (thickness 0.3)))
+  )
   (gr_line (start 156 85) (end 156 73) (layer Edge.Cuts) (width 0.15))
