File: projects/MOTBOX_TOP/motbox_with_promini/motbox_with_promini_v1_2.sch (KiCad schematic (older format))
At the start: 26 parts, among them J1 JST_XH_2pin, J2 Header_3pin_Male, J3 JST_XH_2pin, J4 JST_XH_4pin, J5 JST_XH_2pin, J6 JST_XH_3pin, J7 JST_XH_2pin, P1 Female_Header_12pin, P3 Female_Header_6pin, P5 Female_Header_12pin, U1 LM2576R-5.0, U2 LM393, U3 L293D

Commit message: Touch switch with feedback light changes
Parts:
- J1, J2, J3, J4, J5, J6: Layer (none) -> BOT
Changed lines of the file:
@@
 F 2 "Connector_JST:JST_XH_B02B-XH-A_1x02_P2.50mm_Vertical" H 1500 1750 50  0001 C CNN
 F 3 "~" H 1500 1750 50  0001 C CNN
+F 4 "BOT" H 1500 1750 50  0001 C CNN "Layer"
 	1    1500 1750
 	-1   0    0    1
@@
 F 2 "Connector_JST:JST_XH_B02B-XH-A_1x02_P2.50mm_Vertical" H 1000 6850 50  0001 C CNN
 F 3 "~" H 1000 6850 50  0001 C CNN
+F 4 "BOT" H 1000 6850 50  0001 C CNN "Layer"
 	1    1000 6850
 	-1   0    0    1
@@
 F 2 "Connector_PinHeader_2.54mm:PinHeader_1x03_P2.54mm_Vertical" H 1400 2850 50  0001 C CNN
 F 3 "~" H 1400 2850 50  0001 C CNN
+F 4 "BOT" H 1400 2850 50  0001 C CNN "Layer"
 	1    1400 2850
 	-1   0    0    1
@@
 F 2 "Connector_JST:JST_XH_B02B-XH-A_1x02_P2.50mm_Vertical" H 1400 3600 50  0001 C CNN
 F 3 "~" H 1400 3600 50  0001 C CNN
+F 4 "BOT" H 1400 3600 50  0001 C CNN "Layer"
 	1    1400 3600
 	-1   0    0    1
@@
 F 2 "Connector_JST:JST_XH_B04B-XH-A_1x04_P2.50mm_Vertical" H 1450 4550 50  0001 C CNN
 F 3 "~" H 1450 4550 50  0001 C CNN
+F 4 "BOT" H 1450 4550 50  0001 C CNN "Layer"
 	1    1450 4550
 	-1   0    0    1
@@
 F 2 "Connector_JST:JST_XH_B03B-XH-A_1x03_P2.50mm_Vertical" H 4450 5200 50  0001 C CNN
 F 3 "~" H 4450 5200 50  0001 C CNN
+F 4 "BOT" H 4450 5200 50  0001 C CNN "Layer"
 	1    4450 5200
 	-1   0    0    1
