File: projects/MOTBOX_TOP/motbox_with_promini/motbox_with_promini_v1_4.kicad_pcb (KiCad board)
At the start: 2 copper layers, 81.9 x 65 mm, 27 parts, among them J1 JST_XH_2pin, J2 Header_3pin_Male, J3 JST_XH_2pin, J4 JST_XH_4pin, J5 JST_XH_2pin, J6 JST_XH_3pin, J7 JST_XH_2pin, P1 Female_Header_12pin, P3 Female_Header_12pin, U1 LM2576R-5.0, U2 LM393, U3 L293D

Commit message: Version 1.4
Connections:
- J5 pad 2: Net-(J5-Pad2) -> /A0
- P1 pad 1: /1(Tx) -> (no net)
- P1 pad 2: /0(Rx) -> (no net)
- P3 pad 8: (no net) -> /A0
- R1 pad 2: Net-(J5-Pad2) -> /A0
- U2 pad 3: Net-(J5-Pad2) -> /A0
Routing:
- net /A0: track 0.00 -> 49.7 mm, vias 0 -> 2
- net Net-(J5-Pad2): track 42.1 -> 0.00 mm, vias 2 -> 0
- net GND: vias 28 -> 38
Other:
- board text removed: "TODO : Need to add mounting holes"
