File: projects/MOTBOX_TOP/MOTBOX_TOP_DT045.sch (KiCad schematic (older format))
At the start: 9 parts, among them J1 JST_VH_Housing_2pin, J2 JST_XH_Female_2pin, J3 JST_XH_Female_2pin, J4 JST_XH_Female_3pin, J5 JST_XH_Female_4pin, J6 JST_XH_Female_2pin, J7 JST_XH_Female_2pin, M1 DC Motor, 12V, 5rpm, 37mm dia

Commit message: Top schematics
Changed lines of the file:
@@
 EESchema Schematic File Version 4
+LIBS:MOTBOX_TOP_DT045-cache
 EELAYER 26 0
 EELAYER END
@@
 	1    0    0    -1
 $EndComp
-$Sheet
-S 4700 3000 1500 2000
-U 5CF6A881
-F0 "Motbox_main" 50
-F1 "Motbox_mainsch.sch" 50
-$EndSheet
 $Comp
 L hitesh_custom:JST_Female_3pin J4
@@
 F1 "limit_switch_DT045.sch" 50
 $EndSheet
+$Sheet
+S 4950 3200 1100 1750
+U 5CFE6C87
+F0 "motbox_main" 50
+F1 "motbox_main.sch" 50
+$EndSheet
 $EndSCHEMATC
