File: projects/MOTBOX_TOP/limit_switch_ESE31.sch (KiCad schematic (older format))
At the start: 3 parts, among them J13 Conn_01x03, SW1 ESE31L11T, SW2 ESE31R11T

Commit message: Top schematics
Parts:
- renumbered J13 to J10
Changed lines of the file:
@@
 EESchema Schematic File Version 4
 LIBS:MOTBOX_TOP_ESE31-cache
+LIBS:motbox_with_promini_v1_3-cache
 EELAYER 26 0
 EELAYER END
@@
 With ESE31 Switches and only 3 pin connector
 $Comp
-L Connector_Generic:Conn_01x03 J13
+L Connector_Generic:Conn_01x03 J10
 U 1 1 5CF632DF
 P 3650 2400
-F 0 "J13" V 3616 2212 50  0000 R CNN
+F 0 "J10" V 3616 2212 50  0000 R CNN
 F 1 "Conn_01x03" V 3525 2212 50  0000 R CNN
 F 2 "Connector_Wire:SolderWirePad_1x03_P3.175mm_Drill0.8mm" H 3650 2400 50  0001 C CNN
