File: projects/MOTBOX_TOP/MOTBOX_TOP_ESE31.sch (KiCad schematic (older format))
At the start: 9 parts, among them J1 JST_VH_Housing_2pin, J2 JST_XH_Female_2pin, J3 JST_XH_Female_2pin, J4 JST_XH_Female_3pin, J5 JST_XH_Female_4pin, J6 JST_XH_Female_2pin, J7 JST_XH_Female_2pin, M1 DC Motor, 12V, 5rpm, 37mm dia

Commit message: Top schematics
Changed lines of the file:
@@
 EESchema Schematic File Version 4
 LIBS:MOTBOX_TOP_ESE31-cache
+LIBS:motbox_with_promini_v1_3-cache
 EELAYER 26 0
 EELAYER END
@@
 F0 "IR_RX" 50
 F1 "IR_RX.sch" 50
-$EndSheet
-$Sheet
-S 4850 1100 800  1300
-U 5CC074C2
-F0 "touch_switch" 50
-F1 "touch_switch.sch" 50
 $EndSheet
 $Comp
@@
 	1    0    0    -1
 $EndComp
-$Sheet
-S 4700 3000 1500 2000
-U 5CF6A881
-F0 "Motbox_main" 50
-F1 "Motbox_mainsch.sch" 50
-$EndSheet
 $Comp
 L hitesh_custom:JST_Female_3pin J4
@@
 F1 "limit_switch_ESE31.sch" 50
 $EndSheet
+$Sheet
+S 4200 800  1350 1800
+U 5CFE1655
+F0 "touch_switch" 50
+F1 "touch_switch.sch" 50
+$EndSheet
+$Sheet
+S 4700 3000 1400 2150
+U 5CFE6B0B
+F0 "motbox_main" 50
+F1 "motbox_main.sch" 50
+$EndSheet
 $EndSCHEMATC

Commit message: Changes misc
Parts:
- PWR1: value 12V, 2A SMPS Module -> 12V, 0.5A SMPS Module
Changed lines of the file:
@@
 EESchema Schematic File Version 4
 LIBS:MOTBOX_TOP_ESE31-cache
-LIBS:motbox_with_promini_v1_3-cache
+LIBS:touch_switch_v1_6-cache
+LIBS:motbox_with_promini_v1_71-cache
 EELAYER 26 0
 EELAYER END
@@
 P 2900 5350
 F 0 "PWR1" H 2900 5300 50  0000 L CNN
-F 1 "12V, 2A SMPS Module" H 2900 5650 50  0000 L CNN
+F 1 "12V, 0.5A SMPS Module" H 2900 5650 50  0000 L CNN
 F 2 "" H 2900 5350 50  0001 C CNN
 F 3 "" H 2900 5350 50  0001 C CNN
