File: projects/GP_Boards/Single_gate_adaptor/Single_gate_adaptor/Single_gate_adaptor.sch (KiCad schematic (older format))
At the start: 38 parts, among them J1 Conn_01x15, J2 Conn_01x08, J3 Conn_01x15, J4 Conn_01x08, J5 Conn_01x08, J6 Conn_01x02, U1 74LVC1G97, U10 74LVC1G98, U11 74LVC1G04, U12 74LVC1G14, U13 74LVC1G17, U14 74LVC1G125, U15 74LVC1G86, U16 LMV321, U2 74LVC1G98, U3 74LVC1G04, U4 74LVC1G14, U5 74LVC1G17, U6 74LVC1G125, U7 74LVC1G86, U8 LMV321, U9 74LVC1G97

Commit message: added the GP boards
Parts:
- removed J6: Conn_01x02, Connector_JST:JST_XH_B02B-XH-A_1x02_P2.50mm_Vertical, symbol Connector_Generic:Conn_01x02
- added J6: Conn_01x03, Connector_PinHeader_2.54mm:PinHeader_1x03_P2.54mm_Vertical, symbol Connector_Generic:Conn_01x03
Changed lines of the file:
@@
 EESchema Schematic File Version 4
+LIBS:Single_gate_adaptor-cache
 EELAYER 26 0
 EELAYER END
@@
 Text Label 5725 3920 0    50   ~ 0
 C7
-Text Label 5720 4320 0    50   ~ 0
+Text Label 5730 4520 0    50   ~ 0
 C8
 Text Label 5725 4420 0    50   ~ 0
 C9
-Text Label 5725 4520 0    50   ~ 0
+Text Label 5730 4320 0    50   ~ 0
 C10
-Text Label 5725 4915 0    50   ~ 0
+Text Label 5725 5115 0    50   ~ 0
 C11
 Text Label 5725 5015 0    50   ~ 0
 C12
-Text Label 5725 5115 0    50   ~ 0
+Text Label 5725 4915 0    50   ~ 0
 C13
 Text Label 5730 5805 0    50   ~ 0
@@
 D8
 $Comp
-L Connector_Generic:Conn_01x02 J6
-U 1 1 5D64CAE6
-P 10095 5475
-F 0 "J6" H 10175 5467 50  0000 L CNN
-F 1 "Conn_01x02" H 10175 5376 50  0000 L CNN
-F 2 "Connector_JST:JST_XH_B02B-XH-A_1x02_P2.50mm_Vertical" H 10095 5475 50  0001 C CNN
-F 3 "~" H 10095 5475 50  0001 C CNN
-	1    10095 5475
-	1    0    0    -1
-$EndComp
-$Comp
 L Amplifier_Operational:LMV321 U8
 U 1 1 5D568B67
@@
 Wire Bus Line
 	5620 1430 5620 6005
+$Comp
+L Connector_Generic:Conn_01x03 J6
+U 1 1 5D7523A3
+P 10095 5475
+F 0 "J6" H 10175 5517 50  0000 L CNN
+F 1 "Conn_01x03" H 10175 5426 50  0000 L CNN
+F 2 "Connector_PinHeader_2.54mm:PinHeader_1x03_P2.54mm_Vertical" H 10095 5475 50  0001 C CNN
+F 3 "~" H 10095 5475 50  0001 C CNN
+	1    10095 5475
+	1    0    0    -1
+$EndComp
 $EndSCHEMATC
