File: projects/MOTBOX_TOP/touch_switch/touch_switch_v1_6.kicad_pcb (KiCad board)
At the start: 2 copper layers, 17 x 78 mm, 12 parts, among them J1 Conn_01x04, U1 TTP223

Commit message: New files modified files etc
Parts:
- C1: value 30pF -> 1.2pF
Other:
- board text removed: "LED Display area"
Changed lines of the file:
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@@
   (general
     (thickness 1.6)
-    (drawings 37)
+    (drawings 36)
     (tracks 83)
     (zones 0)
@@
     (39 F.Mask user)
     (40 Dwgs.User user)
-    (41 Cmts.User user)
+    (41 Cmts.User user hide)
     (42 Eco1.User user)
     (43 Eco2.User user)
@@
     (47 F.CrtYd user)
     (48 B.Fab user hide)
-    (49 F.Fab user)
+    (49 F.Fab user hide)
   )
   (setup
@@
       (effects (font (size 1 1) (thickness 0.15)) (justify mirror))
     )
-    (fp_text value 30pF (at 0 -1.43 90) (layer B.Fab)
+    (fp_text value 1.2pF (at 0 -1.43 90) (layer B.Fab)
       (effects (font (size 1 1) (thickness 0.15)) (justify mirror))
     )
@@
     (effects (font (size 1 1) (thickness 0.25)))
   )
-  (gr_text "LED Display \narea" (at 144.388 68.638) (layer Cmts.User)
-    (effects (font (size 1 1) (thickness 0.25)))
-  )
   (gr_text "Touch Panel" (at 145.388 89.138) (layer Cmts.User)
     (effects (font (size 1 1) (thickness 0.25)))
@@
   )
   (dimension 2.000156 (width 0.3) (layer Cmts.User)
-    (gr_text "2.000 mm" (at 127.589378 85.912723 0.7161599455) (layer Cmts.User)
+    (gr_text "2.000 mm" (at 127.553614 79.644011 0.7161599455) (layer Cmts.User)
       (effects (font (size 1.5 1.5) (thickness 0.3)))
     )
-    (feature1 (pts (xy 128.625 88.75) (xy 128.608296 87.413684)))
-    (feature2 (pts (xy 126.625 88.775) (xy 126.608296 87.438684)))
-    (crossbar (pts (xy 126.615626 88.025059) (xy 128.615626 88.000059)))
-    (arrow1a (pts (xy 128.615626 88.000059) (xy 127.49654 88.600514)))
-    (arrow1b (pts (xy 128.615626 88.000059) (xy 127.481881 87.427764)))
-    (arrow2a (pts (xy 126.615626 88.025059) (xy 127.749371 88.597354)))
-    (arrow2b (pts (xy 126.615626 88.025059) (xy 127.734712 87.424604)))
+    (feature1 (pts (xy 128.589236 82.481288) (xy 128.572532 81.144972)))
+    (feature2 (pts (xy 126.589236 82.506288) (xy 126.572532 81.169972)))
+    (crossbar (pts (xy 126.579862 81.756347) (xy 128.579862 81.731347)))
+    (arrow1a (pts (xy 128.579862 81.731347) (xy 127.460776 82.331802)))
+    (arrow1b (pts (xy 128.579862 81.731347) (xy 127.446117 81.159052)))
+    (arrow2a (pts (xy 126.579862 81.756347) (xy 127.713607 82.328642)))
+    (arrow2b (pts (xy 126.579862 81.756347) (xy 127.698948 81.155892)))
   )
   (dimension 2 (width 0.3) (layer Cmts.User)
-    (gr_text "2.000 mm" (at 112.55 86.4) (layer Cmts.User)
+    (gr_text "2.000 mm" (at 112.586058 80.852428) (layer Cmts.User)
       (effects (font (size 1.5 1.5) (thickness 0.3)))
     )
-    (feature1 (pts (xy 113.55 89.3) (xy 113.55 87.913579)))
-    (feature2 (pts (xy 111.55 89.3) (xy 111.55 87.913579)))
-    (crossbar (pts (xy 111.55 88.5) (xy 113.55 88.5)))
-    (arrow1a (pts (xy 113.55 88.5) (xy 112.423496 89.086421)))
-    (arrow1b (pts (xy 113.55 88.5) (xy 112.423496 87.913579)))
-    (arrow2a (pts (xy 111.55 88.5) (xy 112.676504 89.086421)))
-    (arrow2b (pts (xy 111.55 88.5) (xy 112.676504 87.913579)))
+    (feature1 (pts (xy 113.586058 83.752428) (xy 113.586058 82.366007)))
+    (feature2 (pts (xy 111.586058 83.752428) (xy 111.586058 82.366007)))
+    (crossbar (pts (xy 111.586058 82.952428) (xy 113.586058 82.952428)))
+    (arrow1a (pts (xy 113.586058 82.952428) (xy 112.459554 83.538849)))
+    (arrow1b (pts (xy 113.586058 82.952428) (xy 112.459554 82.366007)))
+    (arrow2a (pts (xy 111.586058 82.952428) (xy 112.712562 83.538849)))
+    (arrow2b (pts (xy 111.586058 82.952428) (xy 112.712562 82.366007)))
   )
   (dimension 32.55001 (width 0.3) (layer Cmts.User)
-    (gr_text "32.550 mm" (at 142.519232 111.970118 -89.95599403) (layer Cmts.User)
+    (gr_text "32.50 mm" (at 142.519232 111.970118 -89.95599403) (layer Cmts.User)
       (effects (font (size 1.5 1.5) (thickness 0.3)))
     )
