File: projects/MOTBOX_TOP/touch_switch/touch_switch_v1_6.sch (KiCad schematic (older format))
At the start: 12 parts, among them J1 Conn_01x04, U1 TTP223

Commit message: Changes for improvments
Parts:
- D1: value LED_Small -> LED_RED
- D2: value LED_Small -> LED_BLUE
- D3: value LED_Small -> LED_GREEN
- R1, R2, R3: value 150R -> 150E; footprint Resistor_SMD:R_1206_3216Metric -> Resistor_SMD:R_0603_1608Metric
- S1: footprint Connector_Wire:SolderWirePad_1x01_SMD_5x10mm -> mylib:Touch_pad_with_backlight
Other:
- note added: "As Green was found tobe very bright it is shifted to Switch o/p and Blue was shifted to power indication."
Changed lines of the file:
@@
 EESchema Schematic File Version 4
+LIBS:touch_switch_v1_6-cache
 EELAYER 26 0
 EELAYER END
@@
 P 4800 3650
 F 0 "R1" H 4700 3850 50  0000 L CNN
-F 1 "150R" V 4700 3550 50  0000 L CNN
-F 2 "Resistor_SMD:R_1206_3216Metric" V 4840 3640 50  0001 C CNN
+F 1 "150E" V 4700 3550 50  0000 L CNN
+F 2 "Resistor_SMD:R_0603_1608Metric" V 4840 3640 50  0001 C CNN
 F 3 "~" H 4800 3650 50  0001 C CNN
 	1    4800 3650
@@
 P 5100 3650
 F 0 "R2" H 5150 3850 50  0000 L CNN
-F 1 "150R" V 5200 3550 50  0000 L CNN
-F 2 "Resistor_SMD:R_1206_3216Metric" V 5140 3640 50  0001 C CNN
+F 1 "150E" V 5200 3550 50  0000 L CNN
+F 2 "Resistor_SMD:R_0603_1608Metric" V 5140 3640 50  0001 C CNN
 F 3 "~" H 5100 3650 50  0001 C CNN
 	1    5100 3650
@@
 P 4800 4000
 F 0 "D1" V 4846 3932 50  0000 R CNN
-F 1 "LED_Small" H 4750 4050 50  0000 R CNN
+F 1 "LED_RED" H 4750 4050 50  0000 R CNN
 F 2 "LED_SMD:LED_0603_1608Metric" V 4800 4000 50  0001 C CNN
 F 3 "~" V 4800 4000 50  0001 C CNN
@@
 P 5100 4000
 F 0 "D2" V 5146 3932 50  0000 R CNN
-F 1 "LED_Small" H 5055 3932 50  0000 R CNN
+F 1 "LED_BLUE" H 5055 3932 50  0000 R CNN
 F 2 "LED_SMD:LED_0603_1608Metric" V 5100 4000 50  0001 C CNN
 F 3 "~" V 5100 4000 50  0001 C CNN
@@
 P 5450 3650
 F 0 "R3" H 5500 3850 50  0000 L CNN
-F 1 "150R" V 5550 3550 50  0000 L CNN
-F 2 "Resistor_SMD:R_1206_3216Metric" V 5490 3640 50  0001 C CNN
+F 1 "150E" V 5550 3550 50  0000 L CNN
+F 2 "Resistor_SMD:R_0603_1608Metric" V 5490 3640 50  0001 C CNN
 F 3 "~" H 5450 3650 50  0001 C CNN
 	1    5450 3650
@@
 P 5450 4000
 F 0 "D3" V 5496 3932 50  0000 R CNN
-F 1 "LED_Small" H 5405 3932 50  0000 R CNN
+F 1 "LED_GREEN" H 5405 3932 50  0000 R CNN
 F 2 "LED_SMD:LED_0603_1608Metric" V 5450 4000 50  0001 C CNN
 F 3 "~" V 5450 4000 50  0001 C CNN
@@
 Wire Wire Line
 	6550 4500 7100 4500
+Connection ~ 6550 3400
 $Comp
 L hitesh_custom:Solder_pad S1
@@
 F 0 "S1" H 6700 3450 50  0000 C CNN
 F 1 "Solder_pad" H 6850 3550 50  0000 C CNN
-F 2 "Connector_Wire:SolderWirePad_1x01_SMD_5x10mm" H 6550 3400 50  0001 C CNN
+F 2 "mylib:Touch_pad_with_backlight" H 6550 3400 50  0001 C CNN
 F 3 "" H 6550 3400 50  0001 C CNN
 	1    6550 3400
 	-1   0    0    1
 $EndComp
-Connection ~ 6550 3400
+Text Notes 7050 6650 0    50   ~ 0
+As Green was found tobe very bright it is shifted to Switch o/p and Blue was shifted to power indication.
 $EndSCHEMATC

Commit message: New files modified files etc
Parts:
- C1: value 30pF -> 1.2pF
Other:
- note added: "V1.6 : Required 1.2pF for the correct sensitivity. Refer the document in DOC folder"
- note removed: "As Green was found tobe very bright it is shifted to Switch o/p and Blue was shifted to power indication."
Changed lines of the file:
@@
 P 6550 3900
 F 0 "C1" H 6642 3946 50  0000 L CNN
-F 1 "30pF" H 6642 3855 50  0000 L CNN
+F 1 "1.2pF" H 6642 3855 50  0000 L CNN
 F 2 "Capacitor_SMD:C_0603_1608Metric" H 6550 3900 50  0001 C CNN
 F 3 "~" H 6550 3900 50  0001 C CNN
@@
 $EndComp
 Text Notes 7050 6650 0    50   ~ 0
-As Green was found tobe very bright it is shifted to Switch o/p and Blue was shifted to power indication.
+V1.6 : Required 1.2pF for the correct sensitivity. Refer the document in DOC folder
 $EndSCHEMATC
