File: projects/MOTBOX_TOP/ir_rx_led/ir_rx_led_v1_5.kicad_pcb (KiCad board)
At the start: 2 copper layers, 11.9 x 32 mm, 5 parts, among them J1 Conn_01x03

Commit message: Modified v1_5
Parts:
- added H3: MountingHole, MountingHole:MountingHole_2.2mm_M2_ISO7380, F.Cu at (150.0, 68.0)
- added H4: MountingHole, MountingHole:MountingHole_2.2mm_M2_ISO7380, F.Cu at (150.0, 34.0)
- added H5: MountingHole, MountingHole:MountingHole_2.2mm_M2_ISO7380, F.Cu at (150.0, 42.0)
- added H6: MountingHole, MountingHole:MountingHole_2.2mm_M2_ISO7380, F.Cu at (141.5, 51.0)
- added H7: MountingHole, MountingHole:MountingHole_2.2mm_M2_ISO7380, F.Cu at (150.0, 60.0)
- H1: value MountingHole -> MountingHole
- moved H2 8.00 mm to (133.0, 34.0)
- moved D1 4.18 mm to (137.7, 52.3)
- moved D2 4.05 mm to (137.7, 43.4)
- moved J1 0.47 mm to (133.0, 54.2)
Routing:
- net Net-(D1-Pad1): track 8.29 -> 5.24 mm
- net Net-(D2-Pad1): track 5.82 -> 6.53 mm
Other:
- board size 11.9 x 32 mm -> 23 x 40 mm

Commit message: Changes misc
Parts:
- moved J1 1.91 mm to (134.9, 54.2)
- moved D2 0.66 mm to (138.4, 43.3)
- moved D1 0.66 mm to (138.4, 52.3)
Routing:
- net Net-(D1-Pad1): track 5.24 -> 3.99 mm
- net Net-(D2-Pad1): track 6.53 -> 6.00 mm
Other:
- outline, holes or cut-outs redrawn
- board text added: "IR RX NU V1.5"
- board text removed: "A0"
- board text removed: "A1"
Changed lines of the file:
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@@
   (general
     (thickness 1.6)
-    (drawings 11)
-    (tracks 4)
+    (drawings 14)
+    (tracks 5)
     (zones 0)
     (modules 10)
@@
     (solder_mask_min_width 0.25)
     (aux_axis_origin 0 0)
-    (visible_elements FFFFFF7F)
+    (visible_elements FFFBFF7F)
     (pcbplotparams
       (layerselection 0x010fc_ffffffff)
@@
   )
   (module LED_THT:LED_D5.0mm_Horizontal_O6.35mm_Z9.0mm (layer F.Cu)
-    (at 137.7 43.4 90)
+    (at 138.36 43.34 90)
     (descr "LED, diameter 5.0mm z-position of LED center 3.0mm, 2 pins, diameter 5.0mm z-position of LED center 3.0mm, 2 pins, diameter 5.0mm z-position of LED center 3.0mm, 2 pins, diameter 5.0mm z-position of LED center 9.0mm, 2 pins, diameter 5.0mm z-position of LED center 9.0mm, 2 pins, diameter 5.0mm z-position of LED center 9.0mm, 2 pins")
     (tags "LED diameter 5.0mm z-position of LED center 3.0mm 2 pins diameter 5.0mm z-position of LED center 3.0mm 2 pins diameter 5.0mm z-position of LED center 3.0mm 2 pins diameter 5.0mm z-position of LED center 9.0mm 2 pins diameter 5.0mm z-position of LED center 9.0mm 2 pins diameter 5.0mm z-position of LED center 9.0mm 2 pins")
@@
   )
   (module LED_THT:LED_D5.0mm_Horizontal_O6.35mm_Z9.0mm (layer F.Cu)
-    (at 137.7 52.3 90)
+    (at 138.36 52.34 90)
     (descr "LED, diameter 5.0mm z-position of LED center 3.0mm, 2 pins, diameter 5.0mm z-position of LED center 3.0mm, 2 pins, diameter 5.0mm z-position of LED center 3.0mm, 2 pins, diameter 5.0mm z-position of LED center 9.0mm, 2 pins, diameter 5.0mm z-position of LED center 9.0mm, 2 pins, diameter 5.0mm z-position of LED center 9.0mm, 2 pins")
     (tags "LED diameter 5.0mm z-position of LED center 3.0mm 2 pins diameter 5.0mm z-position of LED center 3.0mm 2 pins diameter 5.0mm z-position of LED center 3.0mm 2 pins diameter 5.0mm z-position of LED center 9.0mm 2 pins diameter 5.0mm z-position of LED center 9.0mm 2 pins diameter 5.0mm z-position of LED center 9.0mm 2 pins")
@@
   )
   (module Connector_Wire:SolderWirePad_1x03_P3.175mm_Drill0.8mm (layer F.Cu)
-    (at 133 54.175 90)
+    (at 134.91 54.215 90)
     (descr "Wire solder connection")
     (tags connector)
@@
     (tags "mounting hole 2.2mm no annular m2 iso7380")
     (attr virtual)
-    (fp_text reference H6 (at 0 2.7) (layer F.SilkS)
+    (fp_text reference H6 (at 1.8 2.61) (layer F.SilkS)
       (effects (font (size 1 1) (thickness 0.15)))
     )
@@
     )
     (pad 1 np_thru_hole circle (at 0 0) (size 2.2 2.2) (drill 2.2) (layers *.Cu *.Mask))
+  )
+  (gr_line (start 130 55.67) (end 130 71) (layer Edge.Cuts) (width 0.1))
+  (gr_line (start 130 31) (end 130.01 46.33) (layer Edge.Cuts) (width 0.1))
+  (gr_line (start 132.5 55.67) (end 130 55.67) (layer Edge.Cuts) (width 0.1))
+  (gr_line (start 132.51 46.33) (end 132.51 55.67) (layer Edge.Cuts) (width 0.1))
+  (gr_line (start 130.01 46.33) (end 132.5 46.33) (layer Edge.Cuts) (width 0.1))
+  (gr_text "IR RX \nNU V1.5" (at 141.45 64.275) (layer F.SilkS)
+    (effects (font (size 1.5 1.5) (thickness 0.3)))
   )
   (gr_line (start 130 51) (end 153 51) (layer Dwgs.User) (width 0.1))
   (gr_line (start 153 71) (end 153 31) (layer Edge.Cuts) (width 0.1))
-  (gr_circle (center 153 60) (end 155.6 61.8) (layer Dwgs.User) (width 0.2))
-  (gr_text A1 (at 137.7 55.3) (layer F.SilkS)
+  (gr_circle (center 151.16 60.04) (end 153.76 61.84) (layer Dwgs.User) (width 0.2))
+  (gr_text G (at 134.88 56.85) (layer F.SilkS)
     (effects (font (size 1.5 1.5) (thickness 0.3)))
   )
-  (gr_text A0 (at 137.7 46.6) (layer F.SilkS)
-    (effects (font (size 1.5 1.5) (thickness 0.3)))
-  )
-  (gr_text G (at 135.5 53.9) (layer F.SilkS)
-    (effects (font (size 1.5 1.5) (thickness 0.3)))
-  )
   (gr_line (start 130 71) (end 153 71) (layer Edge.Cuts) (width 0.1))
-  (gr_line (start 130 31) (end 130 71) (layer Edge.Cuts) (width 0.1))
   (gr_line (start 153 31) (end 130 31) (layer Edge.Cuts) (width 0.1))
-  (gr_circle (center 153 51) (end 155.6 52.8) (layer Dwgs.User) (width 0.2))
-  (gr_circle (center 153 42) (end 155.6 43.8) (layer Dwgs.User) (width 0.2))
-  (segment (start 134.3 52.3) (end 133 51) (width 0.25) (layer B.Cu) (net 2))
-  (segment (start 137.7 52.3) (end 134.3 52.3) (width 0.25) (layer B.Cu) (net 2))
-  (segment (start 137.425 43.4) (end 137.7 43.4) (width 0.25) (layer B.Cu) (net 3))
-  (segment (start 133 47.825) (end 137.425 43.4) (width 0.25) (layer B.Cu) (net 3))
+  (gr_circle (center 151.16 51.04) (end 153.76 52.84) (layer Dwgs.User) (width 0.2))
+  (gr_circle (center 151.16 42.04) (end 153.76 43.84) (layer Dwgs.User) (width 0.2))
+  (segment (start 136.21 52.34) (end 138.36 52.34) (width 0.25) (layer B.Cu) (net 2))
+  (segment (start 134.91 51.04) (end 136.21 52.34) (width 0.25) (layer B.Cu) (net 2))
+  (segment (start 134.985 47.865) (end 134.91 47.865) (width 0.25) (layer B.Cu) (net 3))
+  (segment (start 138.36 44.49) (end 134.985 47.865) (width 0.25) (layer B.Cu) (net 3))
+  (segment (start 138.36 43.34) (end 138.36 44.49) (width 0.25) (layer B.Cu) (net 3))
   (zone (net 1) (net_name "Net-(D1-Pad2)") (layer B.Cu) (hatch edge 0.508)
     (connect_pads (clearance 0.508))

Commit message: Changes for improvments
Parts:
- H1, H2, H3, H4: footprint MountingHole:MountingHole_2.2mm_M2_ISO7380 -> MountingHole:MountingHole_3.2mm_M3_DIN965
- H5, H6, H7: footprint MountingHole:MountingHole_2.2mm_M2_ISO7380 -> MountingHole:MountingHole_2.2mm_M2_DIN965
- moved D2 17.4 mm to (137.8, 60.8)
- moved J1 6.41 mm to (134.3, 47.8), turned to 270 degrees
- moved H5 2.24 mm to (151.0, 40.0)
- moved H7 2.24 mm to (151.0, 62.0)
- moved H1 1.00 mm to (134.0, 68.0)
- moved H2 1.00 mm to (134.0, 34.0)
- moved H3 1.00 mm to (149.0, 68.0)
- moved H4 1.00 mm to (149.0, 34.0)
- moved D1 0.54 mm to (137.8, 52.3)
- moved H6 0.50 mm to (141.0, 51.0)
Routing:
- net Net-(D2-Pad1): track 6.00 -> 8.71 mm
Other:
- board text added: "Hole size and position changes as per the ORG box"
