File: projects/MOTBOX_TOP/ir_rx_led/ir_rx_led_v1_5.sch (KiCad schematic (older format))
At the start: 5 parts, among them J1 Conn_01x03

Commit message: Modified v1_5
Parts:
- added H2, H4, H5, H6, H7: MountingHole, MountingHole:MountingHole_2.2mm_M2_ISO7380, symbol Mechanical:MountingHole
- H1: value MountingHole -> MountingHole
- renumbered H2 to H3
Changed lines of the file:
@@
 L Mechanical:MountingHole H1
 U 1 1 5D352F91
-P 3900 1850
-F 0 "H1" H 4000 1896 50  0000 L CNN
-F 1 "MountingHole" H 4000 1805 50  0000 L CNN
-F 2 "MountingHole:MountingHole_2.2mm_M2_ISO7380" H 3900 1850 50  0001 C CNN
-F 3 "~" H 3900 1850 50  0001 C CNN
-	1    3900 1850
+P 2600 1500
+F 0 "H1" H 2700 1546 50  0000 L CNN
+F 1 " MountingHole" H 2700 1455 50  0000 L CNN
+F 2 "MountingHole:MountingHole_2.2mm_M2_ISO7380" H 2600 1500 50  0001 C CNN
+F 3 "~" H 2600 1500 50  0001 C CNN
+	1    2600 1500
 	1    0    0    -1
 $EndComp
 $Comp
-L Mechanical:MountingHole H2
+L Mechanical:MountingHole H3
 U 1 1 5D352FF3
-P 3900 2750
-F 0 "H2" H 4000 2796 50  0000 L CNN
-F 1 "MountingHole" H 4000 2705 50  0000 L CNN
-F 2 "MountingHole:MountingHole_2.2mm_M2_ISO7380" H 3900 2750 50  0001 C CNN
-F 3 "~" H 3900 2750 50  0001 C CNN
-	1    3900 2750
+P 2600 2200
+F 0 "H3" H 2700 2246 50  0000 L CNN
+F 1 "MountingHole" H 2700 2155 50  0000 L CNN
+F 2 "MountingHole:MountingHole_2.2mm_M2_ISO7380" H 2600 2200 50  0001 C CNN
+F 3 "~" H 2600 2200 50  0001 C CNN
+	1    2600 2200
 	1    0    0    -1
 $EndComp
@@
 Wire Wire Line
 	4500 2450 4500 2700
+$Comp
+L Mechanical:MountingHole H7
+U 1 1 5D42A906
+P 5750 2000
+F 0 "H7" H 5850 2046 50  0000 L CNN
+F 1 "MountingHole" H 5850 1955 50  0000 L CNN
+F 2 "MountingHole:MountingHole_2.2mm_M2_ISO7380" H 5750 2000 50  0001 C CNN
+F 3 "~" H 5750 2000 50  0001 C CNN
+	1    5750 2000
+	1    0    0    -1
+$EndComp
+$Comp
+L Mechanical:MountingHole H5
+U 1 1 5D42A85C
+P 5750 1500
+F 0 "H5" H 5850 1546 50  0000 L CNN
+F 1 "MountingHole" H 5850 1455 50  0000 L CNN
+F 2 "MountingHole:MountingHole_2.2mm_M2_ISO7380" H 5750 1500 50  0001 C CNN
+F 3 "~" H 5750 1500 50  0001 C CNN
+	1    5750 1500
+	1    0    0    -1
+$EndComp
+$Comp
+L Mechanical:MountingHole H2
+U 1 1 5D42B75D
+P 2600 1850
+F 0 "H2" H 2700 1896 50  0000 L CNN
+F 1 "MountingHole" H 2700 1805 50  0000 L CNN
+F 2 "MountingHole:MountingHole_2.2mm_M2_ISO7380" H 2600 1850 50  0001 C CNN
+F 3 "~" H 2600 1850 50  0001 C CNN
+	1    2600 1850
+	1    0    0    -1
+$EndComp
+$Comp
+L Mechanical:MountingHole H4
+U 1 1 5D42B7EB
+P 2600 2500
+F 0 "H4" H 2700 2546 50  0000 L CNN
+F 1 "MountingHole" H 2700 2455 50  0000 L CNN
+F 2 "MountingHole:MountingHole_2.2mm_M2_ISO7380" H 2600 2500 50  0001 C CNN
+F 3 "~" H 2600 2500 50  0001 C CNN
+	1    2600 2500
+	1    0    0    -1
+$EndComp
+$Comp
+L Mechanical:MountingHole H6
+U 1 1 5D42B91F
+P 5750 1750
+F 0 "H6" H 5850 1796 50  0000 L CNN
+F 1 "MountingHole" H 5850 1705 50  0000 L CNN
+F 2 "MountingHole:MountingHole_2.2mm_M2_ISO7380" H 5750 1750 50  0001 C CNN
+F 3 "~" H 5750 1750 50  0001 C CNN
+	1    5750 1750
+	1    0    0    -1
+$EndComp
 $EndSCHEMATC

Commit message: Changes for improvments
Parts:
- H1, H2, H3, H4: footprint MountingHole:MountingHole_2.2mm_M2_ISO7380 -> MountingHole:MountingHole_3.2mm_M3_DIN965
- H5, H6, H7: footprint MountingHole:MountingHole_2.2mm_M2_ISO7380 -> MountingHole:MountingHole_2.2mm_M2_DIN965
Changed lines of the file:
@@
 F 0 "H1" H 2700 1546 50  0000 L CNN
 F 1 " MountingHole" H 2700 1455 50  0000 L CNN
-F 2 "MountingHole:MountingHole_2.2mm_M2_ISO7380" H 2600 1500 50  0001 C CNN
+F 2 "MountingHole:MountingHole_3.2mm_M3_DIN965" H 2600 1500 50  0001 C CNN
 F 3 "~" H 2600 1500 50  0001 C CNN
 	1    2600 1500
@@
 F 0 "H3" H 2700 2246 50  0000 L CNN
 F 1 "MountingHole" H 2700 2155 50  0000 L CNN
-F 2 "MountingHole:MountingHole_2.2mm_M2_ISO7380" H 2600 2200 50  0001 C CNN
+F 2 "MountingHole:MountingHole_3.2mm_M3_DIN965" H 2600 2200 50  0001 C CNN
 F 3 "~" H 2600 2200 50  0001 C CNN
 	1    2600 2200
@@
 F 0 "H7" H 5850 2046 50  0000 L CNN
 F 1 "MountingHole" H 5850 1955 50  0000 L CNN
-F 2 "MountingHole:MountingHole_2.2mm_M2_ISO7380" H 5750 2000 50  0001 C CNN
+F 2 "MountingHole:MountingHole_2.2mm_M2_DIN965" H 5750 2000 50  0001 C CNN
 F 3 "~" H 5750 2000 50  0001 C CNN
 	1    5750 2000
@@
 F 0 "H5" H 5850 1546 50  0000 L CNN
 F 1 "MountingHole" H 5850 1455 50  0000 L CNN
-F 2 "MountingHole:MountingHole_2.2mm_M2_ISO7380" H 5750 1500 50  0001 C CNN
+F 2 "MountingHole:MountingHole_2.2mm_M2_DIN965" H 5750 1500 50  0001 C CNN
 F 3 "~" H 5750 1500 50  0001 C CNN
 	1    5750 1500
@@
 F 0 "H2" H 2700 1896 50  0000 L CNN
 F 1 "MountingHole" H 2700 1805 50  0000 L CNN
-F 2 "MountingHole:MountingHole_2.2mm_M2_ISO7380" H 2600 1850 50  0001 C CNN
+F 2 "MountingHole:MountingHole_3.2mm_M3_DIN965" H 2600 1850 50  0001 C CNN
 F 3 "~" H 2600 1850 50  0001 C CNN
 	1    2600 1850
@@
 F 0 "H4" H 2700 2546 50  0000 L CNN
 F 1 "MountingHole" H 2700 2455 50  0000 L CNN
-F 2 "MountingHole:MountingHole_2.2mm_M2_ISO7380" H 2600 2500 50  0001 C CNN
+F 2 "MountingHole:MountingHole_3.2mm_M3_DIN965" H 2600 2500 50  0001 C CNN
 F 3 "~" H 2600 2500 50  0001 C CNN
 	1    2600 2500
@@
 F 0 "H6" H 5850 1796 50  0000 L CNN
 F 1 "MountingHole" H 5850 1705 50  0000 L CNN
-F 2 "MountingHole:MountingHole_2.2mm_M2_ISO7380" H 5750 1750 50  0001 C CNN
+F 2 "MountingHole:MountingHole_2.2mm_M2_DIN965" H 5750 1750 50  0001 C CNN
 F 3 "~" H 5750 1750 50  0001 C CNN
 	1    5750 1750
