File: projects/occupancy/occupancy_v1_0.sch (KiCad schematic (older format))
At the start: 15 parts, among them J1 Screw_Terminal_01x02, J2 Conn_01x03_Female, J3 Screw_Terminal_01x02, J4 Conn_01x01, K1 JQC-3F-1C-DC5V, Q1 BC547, U1 Easy-Power, U2 LM555

Commit message: layout wIth the GP box dimensions
Parts:
- removed J1, J3: Screw_Terminal_01x02, mylibs:Screw_terminal_2pin_P5mm_width10mm, symbol Connector:Screw_Terminal_01x02
- added H1, H2: MountingHole, MountingHole:MountingHole_3.2mm_M3, symbol Mechanical:MountingHole
- added J1, J3: Conn_01x02, Connector_Wire:SolderWirePad_1x02_P5.08mm_Drill1.5mm, symbol Connector_Generic:Conn_01x02
- J4: footprint Connector_PinHeader_2.54mm:PinHeader_1x01_P2.54mm_Vertical -> Connector_Wire:SolderWirePad_1x01_Drill1.5mm
- Q1: footprint Package_TO_SOT_THT:TO-92_HandSolder -> Package_TO_SOT_THT:TO-92_Wide
Other:
- note added: "As per the GP Box"
Changed lines of the file:
@@
 EESchema Schematic File Version 4
-LIBS:occupancy-cache
 EELAYER 26 0
 EELAYER END
@@
 F 0 "Q1" H 7741 2946 50  0000 L CNN
 F 1 "BC547" H 7741 2855 50  0000 L CNN
-F 2 "Package_TO_SOT_THT:TO-92_HandSolder" H 7750 2825 50  0001 L CIN
+F 2 "Package_TO_SOT_THT:TO-92_Wide" H 7750 2825 50  0001 L CIN
 F 3 "http://www.fairchildsemi.com/ds/BC/BC547.pdf" H 7550 2900 50  0001 L CNN
 	1    7550 2900
@@
 $EndComp
 $Comp
-L Connector:Screw_Terminal_01x02 J1
-U 1 1 5C4739E9
-P 2050 3050
-F 0 "J1" H 1970 2725 50  0000 C CNN
-F 1 "Screw_Terminal_01x02" H 1970 2816 50  0000 C CNN
-F 2 "mylibs:Screw_terminal_2pin_P5mm_width10mm" H 2050 3050 50  0001 C CNN
-F 3 "~" H 2050 3050 50  0001 C CNN
-	1    2050 3050
-	-1   0    0    1
-$EndComp
-$Comp
 L Connector:Conn_01x03_Female J2
 U 1 1 5C473F9C
@@
 	-1   0    0    1
 $EndComp
-Wire Wire Line
-	2250 3050 2250 3100
 $Comp
 L power:GNDREF #PWR0101
@@
 Wire Wire Line
 	2400 2950 2850 2950
-$Comp
-L Connector:Screw_Terminal_01x02 J3
-U 1 1 5C473A8F
+Wire Wire Line
+	8590 4705 2605 4705
+Wire Wire Line
+	2605 4705 2605 3100
+Connection ~ 2605 3100
+Wire Wire Line
+	2605 3100 2850 3100
+Wire Wire Line
+	8050 1755 8050 1950
+Wire Wire Line
+	8050 1950 7950 1950
+Wire Wire Line
+	7950 1755 7950 1845
+Wire Wire Line
+	7950 1845 8590 1845
+Wire Wire Line
+	8590 1845 8590 4705
+Text Notes 7375 6740 0    50   ~ 0
+As per the GP Box
+$Comp
+L Connector_Generic:Conn_01x02 J1
+U 1 1 5DC3D459
+P 2050 3050
+F 0 "J1" H 1970 2725 50  0000 C CNN
+F 1 "Conn_01x02" H 1970 2816 50  0000 C CNN
+F 2 "Connector_Wire:SolderWirePad_1x02_P5.08mm_Drill1.5mm" H 2050 3050 50  0001 C CNN
+F 3 "~" H 2050 3050 50  0001 C CNN
+	1    2050 3050
+	-1   0    0    1
+$EndComp
+Wire Wire Line
+	2250 3050 2250 3100
+Wire Wire Line
+	2250 3100 2605 3100
+Wire Wire Line
+	8150 1755 8150 1950
+$Comp
+L Connector_Generic:Conn_01x02 J3
+U 1 1 5DC413CD
 P 7950 1555
-F 0 "J3" V 7916 1367 50  0000 R CNN
-F 1 "Screw_Terminal_01x02" V 7825 1367 50  0000 R CNN
-F 2 "mylibs:Screw_terminal_2pin_P5mm_width10mm" H 7950 1555 50  0001 C CNN
+F 0 "J3" V 8035 1555 50  0000 R CNN
+F 1 "Conn_01x02" V 8125 1885 50  0000 R CNN
+F 2 "Connector_Wire:SolderWirePad_1x02_P5.08mm_Drill1.5mm" H 7950 1555 50  0001 C CNN
 F 3 "~" H 7950 1555 50  0001 C CNN
 	1    7950 1555
 	0    -1   -1   0
 $EndComp
-Wire Wire Line
-	2250 3100 2605 3100
-Wire Wire Line
-	8590 4705 2605 4705
-Wire Wire Line
-	2605 4705 2605 3100
-Connection ~ 2605 3100
-Wire Wire Line
-	2605 3100 2850 3100
-Wire Wire Line
-	8050 1755 8050 1950
-Wire Wire Line
-	8050 1950 7950 1950
-Wire Wire Line
-	7950 1755 7950 1845
-Wire Wire Line
-	7950 1845 8590 1845
-Wire Wire Line
-	8590 1845 8590 4705
-Wire Wire Line
-	8150 1950 8810 1950
 $Comp
 L Connector_Generic:Conn_01x01 J4
-U 1 1 5DC49214
-P 9010 1950
-F 0 "J4" H 9090 1992 50  0000 L CNN
-F 1 "Conn_01x01" H 9090 1901 50  0000 L CNN
-F 2 "Connector_PinHeader_2.54mm:PinHeader_1x01_P2.54mm_Vertical" H 9010 1950 50  0001 C CNN
-F 3 "~" H 9010 1950 50  0001 C CNN
-	1    9010 1950
-	1    0    0    -1
-$EndComp
+U 1 1 5DC415BB
+P 8150 1555
+F 0 "J4" V 8240 1585 50  0000 R CNN
+F 1 "Conn_01x01" V 8160 1480 50  0000 R CNN
+F 2 "Connector_Wire:SolderWirePad_1x01_Drill1.5mm" H 8150 1555 50  0001 C CNN
+F 3 "~" H 8150 1555 50  0001 C CNN
+	1    8150 1555
+	0    -1   -1   0
+$EndComp
+$Comp
+L Mechanical:MountingHole H1
+U 1 1 5DC41FA0
+P 3370 1145
+F 0 "H1" H 3470 1191 50  0000 L CNN
+F 1 "MountingHole" H 3470 1100 50  0000 L CNN
+F 2 "MountingHole:MountingHole_3.2mm_M3" H 3370 1145 50  0001 C CNN
+F 3 "~" H 3370 1145 50  0001 C CNN
+	1    3370 1145
+	1    0    0    -1
+$EndComp
+$Comp
+L Mechanical:MountingHole H2
+U 1 1 5DC4211C
+P 4590 1100
+F 0 "H2" H 4690 1146 50  0000 L CNN
+F 1 "MountingHole" H 4690 1055 50  0000 L CNN
+F 2 "MountingHole:MountingHole_3.2mm_M3" H 4590 1100 50  0001 C CNN
+F 3 "~" H 4590 1100 50  0001 C CNN
+	1    4590 1100
+	1    0    0    -1
+$EndComp

Commit message: New files modified files etc
Parts:
- removed J1, J3: Conn_01x02, Connector_Wire:SolderWirePad_1x02_P5.08mm_Drill1.5mm, symbol Connector_Generic:Conn_01x02
- added J1, J3, J5: Conn_01x01, Connector_Wire:SolderWirePad_1x01_Drill1.5mm, symbol Connector_Generic:Conn_01x01
- added PCB1: HC-SR501, symbol hitesh_custom:AnyPCB
Connections:
- wire segments 74 -> 68
Changed lines of the file:
@@
 EESchema Schematic File Version 4
+LIBS:occupancy_v1_0-cache
 EELAYER 26 0
 EELAYER END
@@
 	2400 2950 2850 2950
 Wire Wire Line
-	8590 4705 2605 4705
-Wire Wire Line
-	2605 4705 2605 3100
-Connection ~ 2605 3100
-Wire Wire Line
-	2605 3100 2850 3100
-Wire Wire Line
 	8050 1755 8050 1950
 Wire Wire Line
 	8050 1950 7950 1950
-Wire Wire Line
-	7950 1755 7950 1845
-Wire Wire Line
-	7950 1845 8590 1845
-Wire Wire Line
-	8590 1845 8590 4705
 Text Notes 7375 6740 0    50   ~ 0
 As per the GP Box
-$Comp
-L Connector_Generic:Conn_01x02 J1
-U 1 1 5DC3D459
-P 2050 3050
-F 0 "J1" H 1970 2725 50  0000 C CNN
-F 1 "Conn_01x02" H 1970 2816 50  0000 C CNN
-F 2 "Connector_Wire:SolderWirePad_1x02_P5.08mm_Drill1.5mm" H 2050 3050 50  0001 C CNN
-F 3 "~" H 2050 3050 50  0001 C CNN
-	1    2050 3050
-	-1   0    0    1
-$EndComp
 Wire Wire Line
 	2250 3050 2250 3100
 Wire Wire Line
-	2250 3100 2605 3100
-Wire Wire Line
 	8150 1755 8150 1950
-$Comp
-L Connector_Generic:Conn_01x02 J3
-U 1 1 5DC413CD
-P 7950 1555
-F 0 "J3" V 8035 1555 50  0000 R CNN
-F 1 "Conn_01x02" V 8125 1885 50  0000 R CNN
-F 2 "Connector_Wire:SolderWirePad_1x02_P5.08mm_Drill1.5mm" H 7950 1555 50  0001 C CNN
-F 3 "~" H 7950 1555 50  0001 C CNN
-	1    7950 1555
-	0    -1   -1   0
-$EndComp
 $Comp
 L Connector_Generic:Conn_01x01 J4
@@
 	1    0    0    -1
 $EndComp
+$Comp
+L Connector_Generic:Conn_01x01 J3
+U 1 1 5DE8CC50
+P 8050 1555
+F 0 "J3" V 8140 1585 50  0000 R CNN
+F 1 "Conn_01x01" V 8045 2060 50  0000 R CNN
+F 2 "Connector_Wire:SolderWirePad_1x01_Drill1.5mm" H 8050 1555 50  0001 C CNN
+F 3 "~" H 8050 1555 50  0001 C CNN
+	1    8050 1555
+	0    -1   -1   0
+$EndComp
+Wire Wire Line
+	2250 3100 2850 3100
+$Comp
+L Connector_Generic:Conn_01x01 J1
+U 1 1 5DE95A80
+P 2050 2950
+F 0 "J1" V 2140 2980 50  0000 R CNN
+F 1 "Conn_01x01" V 2060 2875 50  0000 R CNN
+F 2 "Connector_Wire:SolderWirePad_1x01_Drill1.5mm" H 2050 2950 50  0001 C CNN
+F 3 "~" H 2050 2950 50  0001 C CNN
+	1    2050 2950
+	-1   0    0    1
+$EndComp
+$Comp
+L Connector_Generic:Conn_01x01 J5
+U 1 1 5DE95A87
+P 2050 3050
+F 0 "J5" V 2140 3080 50  0000 R CNN
+F 1 "Conn_01x01" V 2045 3555 50  0000 R CNN
+F 2 "Connector_Wire:SolderWirePad_1x01_Drill1.5mm" H 2050 3050 50  0001 C CNN
+F 3 "~" H 2050 3050 50  0001 C CNN
+	1    2050 3050
+	-1   0    0    1
+$EndComp
+$Comp
+L hitesh_custom:AnyPCB PCB1
+U 1 1 5DE9A3AB
+P 5950 1265
+F 0 "PCB1" H 6228 1536 50  0000 L CNN
+F 1 "HC-SR501" H 6228 1445 50  0000 L CNN
+F 2 "" H 5950 1265 50  0001 C CNN
+F 3 "" H 5950 1265 50  0001 C CNN
+	1    5950 1265
+	1    0    0    -1
+$EndComp
