File: projects/occupancy/occupancy_v1_1.kicad_pcb (KiCad board)
At the start: 2 copper layers, 53.5 x 59 mm, 18 parts, among them J1 Conn_01x01, J2 Conn_01x03_Female, J3 Conn_01x01, J4 Conn_01x01, J5 Conn_01x01, K1 JQC-3F-1C-DC5V, Q1 BC547, U1 Easy-Power, U2 NE555

Commit message: Cost XLS and v1.1 and changes
Parts:
- removed H1, H2: MountingHole, MountingHole:MountingHole_3.2mm_M3
- C1: value 470uF,16V -> 470uF16V-8X12
- C2: value 0.01uF -> 103-50V
- C3: value 10uF,16V -> 10UF16V-5X11
- J2: value Conn_01x03_Female -> CONN0103
- K1: value JQC-3F-1C-DC5V -> SRD-05VDC-SL-C
- R1: value LDR -> LDR5528
- R2: value 10K -> 10K0.25W
- RV1: value 20K -> 3296W-203
- U2: value NE555 -> NE555P
Other:
- outline, holes or cut-outs redrawn
- board text added: "NU OCC 1.1"
- board text removed: "NU OCC 1.0"
