File: projects/occupancy/occupancy_v1_1.sch (KiCad schematic (older format))
At the start: 19 parts, among them J1 Conn_01x01, J2 Conn_01x03_Female, J3 Conn_01x01, J4 Conn_01x01, J5 Conn_01x01, K1 JQC-3F-1C-DC5V, Q1 BC547, U1 Easy-Power, U2 NE555

Commit message: Cost XLS and v1.1 and changes
Parts:
- removed H1, H2: MountingHole, MountingHole:MountingHole_3.2mm_M3, symbol Mechanical:MountingHole
- removed U2: NE555, Package_DIP:DIP-8_W7.62mm_LongPads, symbol Timer:LM555
- added U2: NE555P, Package_DIP:DIP-8_W7.62mm_LongPads, symbol Timer:NE555
- C1: value 470uF,16V -> 470uF16V-8X12
- C2: value 0.01uF -> 103-50V
- C3: value 10uF,16V -> 10UF16V-5X11
- J2: value Conn_01x03_Female -> CONN0103
- K1: value JQC-3F-1C-DC5V -> SRD-05VDC-SL-C
- R1: value LDR -> LDR5528
- R2: value 10K -> 10K0.25W
- RV1: value 20K -> 3296W-203
Other:
- note added: "As per the GP Box"
- note removed: "As per the GP-05 Box. Rectangle PCB with mounting holes at the end."
Changed lines of the file:
@@
 EESchema Schematic File Version 4
-LIBS:occupancy_v1_0-cache
+LIBS:occupancy_v1_1-cache
 EELAYER 26 0
 EELAYER END
@@
 $EndDescr
 $Comp
-L Timer:LM555 U2
-U 1 1 5C470DB3
-P 6200 3100
-F 0 "U2" H 6500 3450 50  0000 C CNN
-F 1 "NE555" H 6200 3100 50  0000 C CNN
-F 2 "Package_DIP:DIP-8_W7.62mm_LongPads" H 6200 3100 50  0001 C CNN
-F 3 "http://www.ti.com/lit/ds/symlink/lm555.pdf" H 6200 3100 50  0001 C CNN
-	1    6200 3100
-	1    0    0    -1
-$EndComp
-$Comp
 L Diode:1N4001 D1
 U 1 1 5C470ECF
@@
 P 4750 2600
 F 0 "R1" H 4820 2646 50  0000 L CNN
-F 1 "LDR" H 4820 2555 50  0000 L CNN
+F 1 "LDR5528" H 4820 2555 50  0000 L CNN
 F 2 "Resistor_THT:R_Axial_DIN0204_L3.6mm_D1.6mm_P5.08mm_Horizontal" V 4800 2350 50  0001 L CNN
 F 3 "~" H 4750 2550 50  0001 C CNN
@@
 P 7250 3500
 F 0 "C3" H 7341 3546 50  0000 L CNN
-F 1 "10uF,16V" H 7341 3455 50  0000 L CNN
+F 1 "10UF16V-5X11" V 7295 3140 50  0000 L CNN
 F 2 "Capacitor_THT:CP_Radial_D4.0mm_P1.50mm" H 7250 3500 50  0001 C CNN
 F 3 "~" H 7250 3500 50  0001 C CNN
@@
 P 7000 2900
 F 0 "R2" V 6804 2900 50  0000 C CNN
-F 1 "10K" V 6895 2900 50  0000 C CNN
+F 1 "10K0.25W" V 6895 2900 50  0000 C CNN
 F 2 "Resistor_THT:R_Axial_DIN0207_L6.3mm_D2.5mm_P10.16mm_Horizontal" H 7000 2900 50  0001 C CNN
 F 3 "~" H 7000 2900 50  0001 C CNN
@@
 P 4200 3050
 F 0 "C1" H 4291 3096 50  0000 L CNN
-F 1 "470uF,16V" H 4250 2950 50  0000 L CNN
+F 1 "470uF16V-8X12" V 4250 2370 50  0000 L CNN
 F 2 "Capacitor_THT:CP_Radial_D8.0mm_P3.50mm" H 4200 3050 50  0001 C CNN
 F 3 "~" H 4200 3050 50  0001 C CNN
@@
 P 5450 3750
 F 0 "C2" H 5542 3796 50  0000 L CNN
-F 1 "0.01uF" H 5500 3650 50  0000 L CNN
+F 1 "103-50V" H 5500 3650 50  0000 L CNN
 F 2 "Capacitor_THT:C_Disc_D3.0mm_W1.6mm_P2.50mm" H 5450 3750 50  0001 C CNN
 F 3 "~" H 5450 3750 50  0001 C CNN
@@
 P 7850 2250
 F 0 "K1" H 8280 2296 50  0000 L CNN
-F 1 "JQC-3F-1C-DC5V" H 8280 2205 50  0000 L CNN
+F 1 "SRD-05VDC-SL-C" H 8280 2205 50  0000 L CNN
 F 2 "Relay_THT:Relay_SPDT_SANYOU_SRD_Series_Form_C" H 8300 2200 50  0001 L CNN
 F 3 "http://www.sanyourelay.ca/public/products/pdf/SRD.pdf" H 7850 2250 50  0001 C CNN
@@
 P 5250 2550
 F 0 "J2" H 5144 2225 50  0000 C CNN
-F 1 "Conn_01x03_Female" H 5144 2316 50  0000 C CNN
+F 1 "CONN0103" H 5144 2316 50  0000 C CNN
 F 2 "Connector_PinHeader_2.54mm:PinHeader_1x03_P2.54mm_Vertical" H 5250 2550 50  0001 C CNN
 F 3 "~" H 5250 2550 50  0001 C CNN
@@
 P 4750 3650
 F 0 "RV1" H 4680 3696 50  0000 R CNN
-F 1 "20K" H 4680 3605 50  0000 R CNN
+F 1 "3296W-203" V 4680 3605 50  0000 R CNN
 F 2 "Potentiometer_THT:Potentiometer_Bourns_3296W_Vertical" H 4750 3650 50  0001 C CNN
 F 3 "~" H 4750 3650 50  0001 C CNN
@@
 	8050 1950 7950 1950
 Text Notes 7375 6740 0    50   ~ 0
-As per the GP-05 Box. Rectangle PCB with mounting holes at the end.
+As per the GP Box
 Wire Wire Line
 	2250 3050 2250 3100
@@
 $EndComp
 $Comp
-L Mechanical:MountingHole H1
-U 1 1 5DC41FA0
-P 3370 1145
-F 0 "H1" H 3470 1191 50  0000 L CNN
-F 1 "MountingHole" H 3470 1100 50  0000 L CNN
-F 2 "MountingHole:MountingHole_3.2mm_M3" H 3370 1145 50  0001 C CNN
-F 3 "~" H 3370 1145 50  0001 C CNN
-	1    3370 1145
-	1    0    0    -1
-$EndComp
-$Comp
-L Mechanical:MountingHole H2
-U 1 1 5DC4211C
-P 4590 1100
-F 0 "H2" H 4690 1146 50  0000 L CNN
-F 1 "MountingHole" H 4690 1055 50  0000 L CNN
-F 2 "MountingHole:MountingHole_3.2mm_M3" H 4590 1100 50  0001 C CNN
-F 3 "~" H 4590 1100 50  0001 C CNN
-	1    4590 1100
-	1    0    0    -1
-$EndComp
-$Comp
 L Connector_Generic:Conn_01x01 J3
 U 1 1 5DE8CC50
@@
 	1    0    0    -1
 $EndComp
+$Comp
+L Timer:NE555 U2
+U 1 1 5E12DE94
+P 6200 3100
+F 0 "U2" H 6330 3440 50  0000 C CNN
+F 1 "NE555P" H 6190 3115 50  0000 C CNN
+F 2 "Package_DIP:DIP-8_W7.62mm_LongPads" H 6200 3100 50  0001 C CNN
+F 3 "http://www.ti.com/lit/ds/symlink/ne555.pdf" H 6200 3100 50  0001 C CNN
+	1    6200 3100
+	1    0    0    -1
+$EndComp
