File: projects/RF_TX_OCC/rf_tx/rf_tx_v1_0.sch (KiCad schematic (older format))
At the start: 25 parts, among them J1 Conn_01x03, J2 Conn_01x04, J3 Conn_01x01_Female, U1 74LVC1G04, U2 74LVC1G14, U3 74LVC1G86, U4 HT12E

Commit message: New files modified files etc
Parts:
- removed JP11, JP12: Jumper_NO_Small, symbol Device:Jumper_NO_Small
- added BH1: BATTERY_HOLDER, symbol hitesh_custom:BATTERY_HOLDER
- added C2: 1uF, Capacitor_SMD:C_1206_3216Metric, symbol Device:C_Small
- added C3: 100pF, Capacitor_SMD:C_0603_1608Metric, symbol Device:C_Small
- added J4: Conn_01x02, Connector_PinHeader_2.54mm:PinHeader_1x02_P2.54mm_Vertical, symbol Connector_Generic:Conn_01x02
- added U1: 74LVC1G04, Package_TO_SOT_SMD:SOT-23-5, symbol 74xGxx:74LVC1G04
- added U6: BD49ExxG, Package_TO_SOT_SMD:SOT-23-5, symbol Power_Management:BD49ExxG
- C1: footprint (none) -> Capacitor_THT:CP_Radial_D5.0mm_P2.50mm
- J1: footprint (none) -> Connector_PinHeader_2.54mm:PinHeader_1x03_P2.54mm_Vertical
- J2: footprint (none) -> Connector_PinHeader_2.54mm:PinHeader_1x04_P2.54mm_Vertical
- J3: footprint (none) -> Connector_PinHeader_2.54mm:PinHeader_1x01_P2.54mm_Vertical
- JP1, JP10, JP2, JP3, JP4, JP5, JP6, JP7, JP8, JP9: footprint (none) -> Jumper:SolderJumper-2_P1.3mm_Open_RoundedPad1.0x1.5mm
- R1, R2, R3: footprint (none) -> Resistor_SMD:R_0603_1608Metric
- U2: renamed from U1; footprint (none) -> Package_TO_SOT_SMD:SOT-23-5
- U3: renamed from U2; footprint (none) -> Package_TO_SOT_SMD:SOT-23-5
- U4: renamed from U3; footprint (none) -> Package_TO_SOT_SMD:SOT-23-5
- U5: renamed from U4; footprint (none) -> Package_DIP:DIP-18_W7.62mm
Connections:
- net labels added: BAT_LOW_N, SENSOR_LS
- wire segments 69 -> 87
Other:
- moved on the sheet: C1, J1, J2, J3, PCB1, R1, R2, R3, U2, U3, U4, U5
